File: hardware/wordClock.sch (EAGLE design)
At the start: 38 parts, among them J1 SPI_PRG, Q1 MOSFET-PCHANNELSMD, Q2 MOSFET-PCHANNELSMD, Q3 MOSFET-PCHANNELSMD, Q4 MOSFET-PCHANNELSMD, Q5 MOSFET-PCHANNELSMD, Q6 MOSFET-PCHANNELSMD, Q7 MOSFET-PCHANNELSMD, Q8 MOSFET-PCHANNELSMD, U1 ATMEGA328P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

Commit message: update changes to atmega component
Parts:
- removed DS1302: (no value), SparkFun-Connectors:M06LOCK
- removed U1: ATMEGA328P, SparkFun-DigitalIC:ATMEGA328P_PDIP
- added DS1302_RTC: (no value), SparkFun-Connectors:M06FEMALE_LOCK
- added U3: ATMEGA328P, SparkFun-DigitalIC:ATMEGA328_SMT
- Y1: device SparkFun-FreqCtrl:CRYSTALSMD -> SparkFun-FreqCtrl:CRYSTALHC49UV
Connections:
- new net N$3: C3.2, C4.2, C5.2
- new net N$7: C6.2, C7.2, U3.AGND, U3.GND@1, U3.GND@2
- new net SCI: U3.PC5(ADC5/SCL)
- net 5V: now also DS1302_RTC.2, U3.AREF, U3.AVCC, U3.VCC@1, U3.VCC@2; no longer DS1302.2, U1.AREF, U1.AVCC, U1.VCC
- net BLANK: now also U3.PB2(SS/OC1B); no longer U1.PB2(SS/OC1B)
- net CE: now also DS1302_RTC.6; no longer DS1302.6
- net CLK: now also DS1302_RTC.4; no longer DS1302.4
- net GND: now also DS1302_RTC.3; no longer C3.2, C4.2, C5.2, C6.2, C7.2, DS1302.3, U1.GND@1, U1.GND@2
- net HR: now also U3.PC0(ADC0); no longer U1.PC0(ADC0)
- net IO: now also DS1302_RTC.5; no longer DS1302.5
- net M0: now also U3.PD0(RXD); no longer U1.PD0(RXD)
- net M1: now also U3.PD1(TXD); no longer U1.PD1(TXD)
- net M2: now also U3.PD2(INT0); no longer U1.PD2(INT0)
- net M3: now also U3.PD3(INT1); no longer U1.PD3(INT1)
- net M4: now also U3.PD4(XCK/T0); no longer U1.PD4(XCK/T0)
- net M5: now also U3.PD5(T1); no longer U1.PD5(T1)
- net M6: now also U3.PD6(AIN0); no longer U1.PD6(AIN0)
- net M7: now also U3.PD7(AIN1); no longer U1.PD7(AIN1)
- net MIN: now also U3.PC1(ADC1); no longer U1.PC1(ADC1)
- net MISO: now also U3.PB4(MISO); no longer U1.PB4(MISO)
- net N$2: now also U3.PB7(XTAL2/TOSC2); no longer U1.PB7(XTAL2/TOSC2)
- net N$4: now also U3.PB6(XTAL1/TOSC1); no longer U1.PB6(XTAL1/TOSC1)
- net RESET: now also U3.PC6(/RESET); no longer U1.PC6(/RESET)
- net SCL: no longer U1.PC5(ADC5/SCL)
- net SCLK: now also U3.PB5(SCK); no longer U1.PB5(SCK)
- net SDA: now also U3.PC4(ADC4/SDA); no longer U1.PC4(ADC4/SDA)
- net SIN: now also U3.PB3(MOSI/OC2); no longer U1.PB3(MOSI/OC2)
- net VCC1: now also DS1302_RTC.1; no longer DS1302.1
- net XLAT: now also U3.PB1(OC1A); no longer U1.PB1(OC1A)
Other:
- moved on the sheet: C3, C4, C5, C6, C7, R1, Y1

Commit message: Fixed ERC errors and Fixed annotation breaks
Should be all good now, Got broken nets fixed, switched larger usb jack
for a micro.
Parts:
- C1: value (none) -> 10uF
- C2, C3, C4, C5, C8: value (none) -> .1uF
- C6, C7: value (none) -> 22uF
- JP1: value USB_PWR -> USB-MICROB; device SparkFun-Connectors:USBPTH-VERTICAL -> SparkFun-Connectors:USB-MICROB
- SW1: value (none) -> HR
- SW2: value (none) -> MIN
- renumbered HR to SW1, JP4 to COL, MIN to SW2, U$1 to ROW
Connections:
- removed net N$7: C6.2, C7.2, U3.AGND, U3.GND@1, U3.GND@2
- removed net ROW8: COL.9
- removed net ROW9: COL.10
- removed net SCI: U3.PC5(ADC5/SCL)
- net CE: now also U3.PC2(ADC2)
- net CLK: now also U3.PB0(ICP)
- net GND: now also C6.2, C7.2, U3.AGND, U3.GND@1, U3.GND@2
- net IO: now also U3.PC3(ADC3)
- net SCL: now also U3.PC5(ADC5/SCL)
